File: hardware/nanodrone/nanodrone.sch (KiCad schematic (older format))
At the start: 21 parts, among them J1 RTR0, J2 RTR1, J3 RTR2, J4 RTR3, Q1 NUD3124LT1G, Q2 NUD3124LT1G, Q3 NUD3124LT1G, Q4 NUD3124LT1G, U1 Feather

Commit message: Fix pwm connection. Add jlcpcb part numbers
Parts:
- D1: value DGB0 -> DGB1; LCSC Part Number (none) -> C434432
- D2: value DBG1 -> DBG2; LSCS Part Number (none) -> C434432
- Q1, Q2, Q3, Q4: LCSC Part Number (none) -> C8545
- R1, R10, R3, R5, R7, R9: LCSC Part Number (none) -> C17408
- R2, R4, R6, R8: LCSC Part Number (none) -> C17577
Connections:
- net GND: no longer Q1.2 (S), Q2.2 (S), Q3.2 (S), Q4.2 (S)
- net rtrctl0: now also Q1.2 (S)
- net rtrctl1: now also Q2.2 (S)
- net rtrctl2: now also Q3.2 (S)
- net rtrctl3: now also Q4.2 (S)
- net dbg1: now reaches U1.6 (D11)
- net dbg1: now also D1.2 (A)
- net dgb0 renamed dbg2
- net dbg2: now also D2.2 (A); no longer D1.2 (A)
- net dgb1: no longer names the net of U1.4 (D13)
- net dgb1: no longer D2.2 (A)
Changed lines of the file:
@@
 Title "Nano Drone"
 Date "2021-09-08"
-Rev "REV A"
+Rev "REV B"
 Comp ""
 Comment1 "Mini drone based on and Arduino Nano BLE Sense"
@@
 $EndComp
 $Comp
-L power:GND #PWR0101
-U 1 1 613A12F9
-P 4350 4050
-F 0 "#PWR0101" H 4350 3800 50  0001 C CNN
-F 1 "GND" H 4355 3877 50  0000 C CNN
-F 2 "" H 4350 4050 50  0001 C CNN
-F 3 "" H 4350 4050 50  0001 C CNN
-	1    4350 4050
-	1    0    0    -1
-$EndComp
-$Comp
 L power:+BATT #PWR0102
 U 1 1 613A3525
@@
 F 3 "~" H 3950 4000 50  0001 C CNN
 F 4 "RMCF0805FT10K0TR-ND" H 3950 4000 50  0001 C CNN "Digi-Key_PN"
+F 5 "C17408" H 3950 4000 50  0001 C CNN "LCSC Part Number"
 	1    3950 4000
 	1    0    0    -1
@@
 F 3 "~" H 4350 3300 50  0001 C CNN
 F 4 "764-1510-2-ND" H 4350 3300 50  0001 C CNN "Digi-Key_PN"
+F 5 "C17577" H 4350 3300 50  0001 C CNN "LCSC Part Number"
 	1    4350 3300
 	1    0    0    -1
@@
 Wire Wire Line
 	4350 3150 4350 3050
-Wire Wire Line
-	4350 3950 4350 4050
-Wire Wire Line
-	3950 4150 3950 4350
-$Comp
-L power:GND #PWR0107
-U 1 1 613BD558
-P 5700 4050
-F 0 "#PWR0107" H 5700 3800 50  0001 C CNN
-F 1 "GND" H 5705 3877 50  0000 C CNN
-F 2 "" H 5700 4050 50  0001 C CNN
-F 3 "" H 5700 4050 50  0001 C CNN
-	1    5700 4050
-	1    0    0    -1
-$EndComp
 $Comp
 L power:+BATT #PWR0108
@@
 F 3 "~" H 5300 4000 50  0001 C CNN
 F 4 "RMCF0805FT10K0TR-ND" H 5300 4000 50  0001 C CNN "Digi-Key_PN"
+F 5 "C17408" H 5300 4000 50  0001 C CNN "LCSC Part Number"
 	1    5300 4000
 	1    0    0    -1
@@
 F 3 "~" H 5700 3300 50  0001 C CNN
 F 4 "764-1510-2-ND" H 5700 3300 50  0001 C CNN "Digi-Key_PN"
+F 5 "C17577" H 5700 3300 50  0001 C CNN "LCSC Part Number"
 	1    5700 3300
 	1    0    0    -1
@@
 Wire Wire Line
 	5700 3150 5700 3050
-Wire Wire Line
-	5700 3950 5700 4050
-Wire Wire Line
-	5300 4150 5300 4350
-$Comp
-L power:GND #PWR0110
-U 1 1 613C3034
-P 7050 4050
-F 0 "#PWR0110" H 7050 3800 50  0001 C CNN
-F 1 "GND" H 7055 3877 50  0000 C CNN
-F 2 "" H 7050 4050 50  0001 C CNN
-F 3 "" H 7050 4050 50  0001 C CNN
-	1    7050 4050
-	1    0    0    -1
-$EndComp
 $Comp
 L power:+BATT #PWR0111
@@
 F 3 "~" H 6650 4000 50  0001 C CNN
 F 4 "RMCF0805FT10K0TR-ND" H 6650 4000 50  0001 C CNN "Digi-Key_PN"
+F 5 "C17408" H 6650 4000 50  0001 C CNN "LCSC Part Number"
 	1    6650 4000
 	1    0    0    -1
@@
 F 3 "~" H 7050 3300 50  0001 C CNN
 F 4 "764-1510-2-ND" H 7050 3300 50  0001 C CNN "Digi-Key_PN"
+F 5 "C17577" H 7050 3300 50  0001 C CNN "LCSC Part Number"
 	1    7050 3300
 	1    0    0    -1
@@
 Wire Wire Line
 	7050 3150 7050 3050
-Wire Wire Line
-	7050 3950 7050 4050
-Wire Wire Line
-	6650 4150 6650 4350
-$Comp
-L power:GND #PWR0113
-U 1 1 613C80E8
-P 8400 4050
-F 0 "#PWR0113" H 8400 3800 50  0001 C CNN
-F 1 "GND" H 8405 3877 50  0000 C CNN
-F 2 "" H 8400 4050 50  0001 C CNN
-F 3 "" H 8400 4050 50  0001 C CNN
-	1    8400 4050
-	1    0    0    -1
-$EndComp
 $Comp
 L power:+BATT #PWR0114
@@
 F 3 "~" H 8000 4000 50  0001 C CNN
 F 4 "RMCF0805FT10K0TR-ND" H 8000 4000 50  0001 C CNN "Digi-Key_PN"
+F 5 "C17408" H 8000 4000 50  0001 C CNN "LCSC Part Number"
 	1    8000 4000
 	1    0    0    -1
@@
 F 3 "~" H 8400 3300 50  0001 C CNN
 F 4 "764-1510-2-ND" H 8400 3300 50  0001 C CNN "Digi-Key_PN"
+F 5 "C17577" H 8400 3300 50  0001 C CNN "LCSC Part Number"
 	1    8400 3300
 	1    0    0    -1
@@
 	8400 3150 8400 3050
 Wire Wire Line
-	8400 3950 8400 4050
-Wire Wire Line
-	8000 4150 8000 4350
-Wire Wire Line
 	4350 3500 4550 3500
 Connection ~ 4350 3500
@@
 Wire Wire Line
 	8400 3500 8400 3450
-Text Label 3950 4350 2    50   ~ 0
-rtrctl0
-Text Label 5300 4350 2    50   ~ 0
-rtrctl1
-Text Label 6650 4350 2    50   ~ 0
-rtrctl2
-Text Label 8000 4350 2    50   ~ 0
-rtrctl3
 Text Label 4550 3500 0    50   ~ 0
 rtr0
@@
 P 6150 5300
 F 0 "D1" V 6250 5450 50  0000 C CNN
-F 1 "DGB0" V 6150 5450 50  0000 C CNN
+F 1 "DGB1" V 6150 5450 50  0000 C CNN
 F 2 "LED_SMD:LED_0805_2012Metric" H 6150 5300 50  0001 C CNN
 F 3 "~" H 6150 5300 50  0001 C CNN
 F 4 "475-1410-2-ND" V 6150 5300 50  0001 C CNN "Digi-Key_PN"
+F 5 "C434432" V 6150 5300 50  0001 C CNN "LCSC Part Number"
 	1    6150 5300
 	0    -1   -1   0
@@
 P 6600 5300
 F 0 "D2" V 6700 5450 50  0000 C CNN
-F 1 "DBG1" V 6600 5450 50  0000 C CNN
+F 1 "DBG2" V 6600 5450 50  0000 C CNN
 F 2 "LED_SMD:LED_0805_2012Metric_Pad1.15x1.40mm_HandSolder" H 6600 5300 50  0001 C CNN
 F 3 "~" H 6600 5300 50  0001 C CNN
 F 4 "475-1410-2-ND" V 6600 5300 50  0001 C CNN "Digi-Key_PN"
+F 5 "C434432" V 6600 5300 50  0001 C CNN "LSCS Part Number"
 	1    6600 5300
 	0    -1   -1   0
@@
 F 3 "~" H 6150 5700 50  0001 C CNN
 F 4 "P100ATR-ND" H 6150 5700 50  0001 C CNN "Digi-Key_PN"
+F 5 "C17408" H 6150 5700 50  0001 C CNN "LCSC Part Number"
 	1    6150 5700
 	1    0    0    -1
@@
 F 3 "~" H 6600 5700 50  0001 C CNN
 F 4 "P100ATR-ND" H 6600 5700 50  0001 C CNN "Digi-Key_PN"
+F 5 "C17408" H 6600 5700 50  0001 C CNN "LCSC Part Number"
 	1    6600 5700
 	1    0    0    -1
@@
 Wire Wire Line
 	6150 5150 6150 5000
-Text Label 6150 5000 0    50   ~ 0
-dgb0
-Wire Wire Line
-	2550 4550 2700 4550
-Text Label 2700 4550 0    50   ~ 0
-dgb0
 Text Notes 9300 2750 0    50   ~ 0
 Rotor Ports
@@
 Status / Debug LEDs
 Wire Wire Line
-	2550 4650 2700 4650
-Wire Wire Line
 	6600 5150 6600 5000
-Text Label 2700 4650 0    50   ~ 0
-dgb1
-Text Label 6600 5000 0    50   ~ 0
-dgb1
 Wire Wire Line
 	2550 4050 2700 4050
@@
 P 4350 3750
 F 0 "Q1" H 4455 3796 50  0000 L CNN
-F 1 "NUD3124LT1G" H 4455 3705 50  0000 L CNN
+F 1 "NUD3124LT1G" H 4455 3705 50  0001 L CNN
 F 2 "Package_TO_SOT_SMD:SOT-23" H 4350 4200 50  0001 C CNN
 F 3 "https://www.onsemi.com/pdf/datasheet/nud3124-d.pdf" H 4350 4200 50  0001 C CNN
 F 4 "NUD3124LT1GOSTR-ND" H 4350 3750 50  0001 C CNN "Digi-Key_PN"
+F 5 "C8545" H 4350 3750 50  0001 C CNN "LCSC Part Number"
 	1    4350 3750
 	1    0    0    -1
@@
 P 5700 3750
 F 0 "Q2" H 5805 3796 50  0000 L CNN
-F 1 "NUD3124LT1G" H 5805 3705 50  0000 L CNN
+F 1 "NUD3124LT1G" H 5805 3705 50  0001 L CNN
 F 2 "Package_TO_SOT_SMD:SOT-23" H 5700 4200 50  0001 C CNN
 F 3 "https://www.onsemi.com/pdf/datasheet/nud3124-d.pdf" H 5700 4200 50  0001 C CNN
 F 4 "NUD3124LT1GOSTR-ND" H 5700 3750 50  0001 C CNN "Digi-Key_PN"
+F 5 "C8545" H 5700 3750 50  0001 C CNN "LCSC Part Number"
 	1    5700 3750
 	1    0    0    -1
@@
 P 7050 3750
 F 0 "Q3" H 7155 3796 50  0000 L CNN
-F 1 "NUD3124LT1G" H 7155 3705 50  0000 L CNN
+F 1 "NUD3124LT1G" H 7155 3705 50  0001 L CNN
 F 2 "Package_TO_SOT_SMD:SOT-23" H 7050 4200 50  0001 C CNN
 F 3 "https://www.onsemi.com/pdf/datasheet/nud3124-d.pdf" H 7050 4200 50  0001 C CNN
 F 4 "NUD3124LT1GOSTR-ND" H 7050 3750 50  0001 C CNN "Digi-Key_PN"
+F 5 "C8545" H 7050 3750 50  0001 C CNN "LCSC Part Number"
 	1    7050 3750
 	1    0    0    -1
@@
 P 8400 3750
 F 0 "Q4" H 8505 3796 50  0000 L CNN
-F 1 "NUD3124LT1G" H 8505 3705 50  0000 L CNN
+F 1 "NUD3124LT1G" H 8505 3705 50  0001 L CNN
 F 2 "Package_TO_SOT_SMD:SOT-23" H 8400 4200 50  0001 C CNN
 F 3 "https://www.onsemi.com/pdf/datasheet/nud3124-d.pdf" H 8400 4200 50  0001 C CNN
 F 4 "NUD3124LT1GOSTR-ND" H 8400 3750 50  0001 C CNN "Digi-Key_PN"
+F 5 "C8545" H 8400 3750 50  0001 C CNN "LCSC Part Number"
 	1    8400 3750
 	1    0    0    -1
@@
 Wire Notes Line
 	7700 4450 7700 2800
+Wire Wire Line
+	3950 4150 3950 4300
+Wire Wire Line
+	3950 4300 4350 4300
+Wire Wire Line
+	4350 4300 4350 3950
+Wire Wire Line
+	5300 4150 5300 4300
+Wire Wire Line
+	5300 4300 5700 4300
+Wire Wire Line
+	5700 4300 5700 3950
+Wire Wire Line
+	6650 4150 6650 4300
+Wire Wire Line
+	6650 4300 7050 4300
+Wire Wire Line
+	7050 4300 7050 3950
+Wire Wire Line
+	8000 4150 8000 4300
+Wire Wire Line
+	8000 4300 8400 4300
+Wire Wire Line
+	8400 4300 8400 3950
+Wire Wire Line
+	3950 4300 3900 4300
+Connection ~ 3950 4300
+Text Label 3900 4300 2    50   ~ 0
+rtrctl0
+Wire Wire Line
+	5300 4300 5250 4300
+Connection ~ 5300 4300
+Text Label 5250 4300 2    50   ~ 0
+rtrctl1
+Wire Wire Line
+	6650 4300 6600 4300
+Connection ~ 6650 4300
+Text Label 6600 4300 2    50   ~ 0
+rtrctl2
+Wire Wire Line
+	8000 4300 7950 4300
+Connection ~ 8000 4300
+Text Label 7950 4300 2    50   ~ 0
+rtrctl3
+Wire Wire Line
+	2550 4450 2700 4450
+Wire Wire Line
+	2550 4550 2700 4550
+Text Label 2700 4450 0    50   ~ 0
+dbg1
+Text Label 2700 4550 0    50   ~ 0
+dbg2
+Text Label 6150 5000 0    50   ~ 0
+dbg1
+Text Label 6600 5000 0    50   ~ 0
+dbg2
 $EndSCHEMATC

Commit message: Rev C
Parts:
- removed Q1, Q2, Q3, Q4: NUD3124LT1G, Package_TO_SOT_SMD:SOT-23, symbol transistors:NUD3124LT1G
- removed R3, R7: 10k, Resistor_SMD:R_0805_2012Metric_Pad1.20x1.40mm_HandSolder, symbol Device:R
- added Q1, Q2, Q3, Q4: SI2302, Package_TO_SOT_SMD:SOT-23, symbol Transistor_FET:2N7002E
- added R11, R14: 25, Resistor_SMD:R_0805_2012Metric_Pad1.20x1.40mm_HandSolder, symbol Device:R
- added R12: 12k, Resistor_SMD:R_0805_2012Metric_Pad1.20x1.40mm_HandSolder, symbol Device:R
- added R13, R2, R9: 4.64k, Resistor_SMD:R_0805_2012Metric_Pad1.20x1.40mm_HandSolder, symbol Device:R
- R1: value 10k -> 12k; Digi-Key_PN RMCF0805FT10K0TR-ND -> (none); LCSC (none) -> C17444; LCSC Part Number C17408 -> (none)
- R4, R8: value 25 -> 12k; Digi-Key_PN 764-1510-2-ND -> (none); LCSC (none) -> C17444; LCSC Part Number C17577 -> (none)
- R5: value 10k -> 4.64k; Digi-Key_PN RMCF0805FT10K0TR-ND -> (none); LCSC (none) -> C170914; LCSC Part Number C17408 -> (none)
- renumbered R2 to R3, R9 to R7
Connections:
- net +3V3: now also R4.1, R8.1, R12.1; no longer R5.1
- net +BATT: now also R11.1, R14.1; no longer R4.1, R8.1
- net GND: now also Q1.2 (S), Q2.2 (S), Q3.2 (S), Q4.2 (S)
- net rtr0: now also Q1.3 (D)
- net rtr1: now also R6.2, Q2.3 (D); no longer R4.2
- net rtr2: now also Q3.3 (D), R11.2; no longer R6.2
- net rtr3: now also Q4.3 (D), R14.2; no longer R8.2
- net rtrctl0: now also R2.2; no longer R1.2
- net rtrctl1: now also R5.2
- net rtrctl2: now also R9.2; no longer R5.2
- net rtrctl3: now also R13.2
- new net: Q1.1 (G), R1.2, R2.1
- new net: Q2.1 (G), R4.2, R5.1
- new net: Q3.1 (G), R8.2, R9.1
- new net: Q4.1 (G), R12.2, R13.1
Other:
- moved on the sheet: R1

Commit message: Rev D
Connections:
- net rtrctl0 is gone; now on net GND: R2.2, U1.10 (D5)
- net rtrctl1 is gone; now on net GND: R5.2, U1.9 (D6)
- net rtrctl2 is gone; now on net GND: R9.2, U1.8 (D9)
- net rtrctl3 is gone; now on net GND: R13.2, U1.7 (D10)
Other:
- moved on the sheet: D1, D2, R10, R7
Changed lines of the file:
@@
 L Device:LED D1
 U 1 1 613AA8FC
-P 6150 5300
-F 0 "D1" V 6250 5450 50  0000 C CNN
-F 1 "DGB1" V 6150 5450 50  0000 C CNN
-F 2 "LED_SMD:LED_0805_2012Metric" H 6150 5300 50  0001 C CNN
-F 3 "~" H 6150 5300 50  0001 C CNN
-F 4 "475-1410-2-ND" V 6150 5300 50  0001 C CNN "Digi-Key_PN"
-F 5 "C434432" V 6150 5300 50  0001 C CNN "LCSC Part Number"
-	1    6150 5300
+P 5350 5700
+F 0 "D1" V 5450 5850 50  0000 C CNN
+F 1 "DGB1" V 5350 5850 50  0000 C CNN
+F 2 "LED_SMD:LED_0805_2012Metric" H 5350 5700 50  0001 C CNN
+F 3 "~" H 5350 5700 50  0001 C CNN
+F 4 "475-1410-2-ND" V 5350 5700 50  0001 C CNN "Digi-Key_PN"
+F 5 "C434432" V 5350 5700 50  0001 C CNN "LCSC Part Number"
+	1    5350 5700
 	0    -1   -1   0
 $EndComp
@@
 L Device:LED D2
 U 1 1 613AAEC3
-P 6600 5300
-F 0 "D2" V 6700 5450 50  0000 C CNN
-F 1 "DBG2" V 6600 5450 50  0000 C CNN
-F 2 "LED_SMD:LED_0805_2012Metric_Pad1.15x1.40mm_HandSolder" H 6600 5300 50  0001 C CNN
-F 3 "~" H 6600 5300 50  0001 C CNN
-F 4 "475-1410-2-ND" V 6600 5300 50  0001 C CNN "Digi-Key_PN"
-F 5 "C434432" V 6600 5300 50  0001 C CNN "LSCS Part Number"
-	1    6600 5300
+P 5800 5700
+F 0 "D2" V 5900 5850 50  0000 C CNN
+F 1 "DBG2" V 5800 5850 50  0000 C CNN
+F 2 "LED_SMD:LED_0805_2012Metric_Pad1.15x1.40mm_HandSolder" H 5800 5700 50  0001 C CNN
+F 3 "~" H 5800 5700 50  0001 C CNN
+F 4 "475-1410-2-ND" V 5800 5700 50  0001 C CNN "Digi-Key_PN"
+F 5 "C434432" V 5800 5700 50  0001 C CNN "LSCS Part Number"
+	1    5800 5700
 	0    -1   -1   0
 $EndComp
@@
 L Device:R R7
 U 1 1 613AC424
-P 6150 5700
-F 0 "R7" H 6000 5800 50  0000 C CNN
-F 1 "100" H 6000 5700 50  0000 C CNN
-F 2 "Resistor_SMD:R_0805_2012Metric_Pad1.15x1.40mm_HandSolder" V 6080 5700 50  0001 C CNN
-F 3 "~" H 6150 5700 50  0001 C CNN
-F 4 "P100ATR-ND" H 6150 5700 50  0001 C CNN "Digi-Key_PN"
-F 5 "C17408" H 6150 5700 50  0001 C CNN "LCSC Part Number"
-	1    6150 5700
+P 5350 6100
+F 0 "R7" H 5200 6200 50  0000 C CNN
+F 1 "100" H 5200 6100 50  0000 C CNN
+F 2 "Resistor_SMD:R_0805_2012Metric_Pad1.15x1.40mm_HandSolder" V 5280 6100 50  0001 C CNN
+F 3 "~" H 5350 6100 50  0001 C CNN
+F 4 "P100ATR-ND" H 5350 6100 50  0001 C CNN "Digi-Key_PN"
+F 5 "C17408" H 5350 6100 50  0001 C CNN "LCSC Part Number"
+	1    5350 6100
 	1    0    0    -1
 $EndComp
@@
 L Device:R R10
 U 1 1 613ACDB5
-P 6600 5700
-F 0 "R10" H 6450 5800 50  0000 C CNN
-F 1 "100" H 6450 5700 50  0000 C CNN
-F 2 "Resistor_SMD:R_0805_2012Metric_Pad1.15x1.40mm_HandSolder" V 6530 5700 50  0001 C CNN
-F 3 "~" H 6600 5700 50  0001 C CNN
-F 4 "P100ATR-ND" H 6600 5700 50  0001 C CNN "Digi-Key_PN"
-F 5 "C17408" H 6600 5700 50  0001 C CNN "LCSC Part Number"
-	1    6600 5700
-	1    0    0    -1
-$EndComp
-Wire Wire Line
-	6150 5550 6150 5450
-Wire Wire Line
-	6600 5550 6600 5450
+P 5800 6100
+F 0 "R10" H 5650 6200 50  0000 C CNN
+F 1 "100" H 5650 6100 50  0000 C CNN
+F 2 "Resistor_SMD:R_0805_2012Metric_Pad1.15x1.40mm_HandSolder" V 5730 6100 50  0001 C CNN
+F 3 "~" H 5800 6100 50  0001 C CNN
+F 4 "P100ATR-ND" H 5800 6100 50  0001 C CNN "Digi-Key_PN"
+F 5 "C17408" H 5800 6100 50  0001 C CNN "LCSC Part Number"
+	1    5800 6100
+	1    0    0    -1
+$EndComp
+Wire Wire Line
+	5350 5950 5350 5850
+Wire Wire Line
+	5800 5950 5800 5850
 $Comp
 L power:GND #PWR01
 U 1 1 613B4116
-P 6150 5950
-F 0 "#PWR01" H 6150 5700 50  0001 C CNN
-F 1 "GND" H 6155 5777 50  0000 C CNN
-F 2 "" H 6150 5950 50  0001 C CNN
-F 3 "" H 6150 5950 50  0001 C CNN
-	1    6150 5950
+P 5350 6350
+F 0 "#PWR01" H 5350 6100 50  0001 C CNN
+F 1 "GND" H 5355 6177 50  0000 C CNN
+F 2 "" H 5350 6350 50  0001 C CNN
+F 3 "" H 5350 6350 50  0001 C CNN
+	1    5350 6350
 	1    0    0    -1
 $EndComp
@@
 L power:GND #PWR02
 U 1 1 613B4CBB
-P 6600 5950
-F 0 "#PWR02" H 6600 5700 50  0001 C CNN
-F 1 "GND" H 6605 5777 50  0000 C CNN
-F 2 "" H 6600 5950 50  0001 C CNN
-F 3 "" H 6600 5950 50  0001 C CNN
-	1    6600 5950
-	1    0    0    -1
-$EndComp
-Wire Wire Line
-	6150 5950 6150 5850
-Wire Wire Line
-	6600 5950 6600 5850
-Wire Wire Line
-	6150 5150 6150 5000
+P 5800 6350
+F 0 "#PWR02" H 5800 6100 50  0001 C CNN
+F 1 "GND" H 5805 6177 50  0000 C CNN
+F 2 "" H 5800 6350 50  0001 C CNN
+F 3 "" H 5800 6350 50  0001 C CNN
+	1    5800 6350
+	1    0    0    -1
+$EndComp
+Wire Wire Line
+	5350 6350 5350 6250
+Wire Wire Line
+	5800 6350 5800 6250
+Wire Wire Line
+	5350 5550 5350 5400
 Text Notes 9300 2750 0    50   ~ 0
 Rotor Ports
-Text Notes 5850 4700 0    50   ~ 0
+Text Notes 5050 5100 0    50   ~ 0
 Status / Debug LEDs
 Wire Wire Line
-	6600 5150 6600 5000
+	5800 5550 5800 5400
 Wire Wire Line
 	2550 4050 2700 4050
@@
 	3000 2450 1500 2450
 Wire Notes Line
-	5850 4750 6950 4750
-Wire Notes Line
-	6950 4750 6950 6200
-Wire Notes Line
-	6950 6200 5850 6200
-Wire Notes Line
-	5850 6200 5850 4750
+	5050 5150 6150 5150
+Wire Notes Line
+	6150 5150 6150 6600
+Wire Notes Line
+	6150 6600 5050 6600
+Wire Notes Line
+	5050 6600 5050 5150
 Wire Notes Line
 	9300 2800 9300 3950
@@
 Text Label 2700 4550 0    50   ~ 0
 dbg2
-Text Label 6150 5000 0    50   ~ 0
+Text Label 5350 5400 0    50   ~ 0
 dbg1
-Text Label 6600 5000 0    50   ~ 0
+Text Label 5800 5400 0    50   ~ 0
 dbg2
 $Comp
@@
 L power:GND #PWR03
 U 1 1 6196904D
-P 4350 4150
-F 0 "#PWR03" H 4350 3900 50  0001 C CNN
-F 1 "GND" H 4355 3977 50  0000 C CNN
-F 2 "" H 4350 4150 50  0001 C CNN
-F 3 "" H 4350 4150 50  0001 C CNN
-	1    4350 4150
-	1    0    0    -1
-$EndComp
-Wire Wire Line
-	4350 4150 4350 3950
+P 4350 4400
+F 0 "#PWR03" H 4350 4150 50  0001 C CNN
+F 1 "GND" H 4355 4227 50  0000 C CNN
+F 2 "" H 4350 4400 50  0001 C CNN
+F 3 "" H 4350 4400 50  0001 C CNN
+	1    4350 4400
+	1    0    0    -1
+$EndComp
 Wire Wire Line
 	3750 4300 3900 4300
@@
 L power:GND #PWR06
 U 1 1 619BFE47
-P 5700 4150
-F 0 "#PWR06" H 5700 3900 50  0001 C CNN
-F 1 "GND" H 5705 3977 50  0000 C CNN
-F 2 "" H 5700 4150 50  0001 C CNN
-F 3 "" H 5700 4150 50  0001 C CNN
-	1    5700 4150
-	1    0    0    -1
-$EndComp
-Wire Wire Line
-	5700 4150 5700 3950
+P 5700 4400
+F 0 "#PWR06" H 5700 4150 50  0001 C CNN
+F 1 "GND" H 5705 4227 50  0000 C CNN
+F 2 "" H 5700 4400 50  0001 C CNN
+F 3 "" H 5700 4400 50  0001 C CNN
+	1    5700 4400
+	1    0    0    -1
+$EndComp
 Wire Wire Line
 	5100 4300 5250 4300
@@
 L power:GND #PWR09
 U 1 1 619C620B
-P 7050 4150
-F 0 "#PWR09" H 7050 3900 50  0001 C CNN
-F 1 "GND" H 7055 3977 50  0000 C CNN
-F 2 "" H 7050 4150 50  0001 C CNN
-F 3 "" H 7050 4150 50  0001 C CNN
-	1    7050 4150
-	1    0    0    -1
-$EndComp
-Wire Wire Line
-	7050 4150 7050 3950
+P 7050 4400
+F 0 "#PWR09" H 7050 4150 50  0001 C CNN
+F 1 "GND" H 7055 4227 50  0000 C CNN
+F 2 "" H 7050 4400 50  0001 C CNN
+F 3 "" H 7050 4400 50  0001 C CNN
+	1    7050 4400
+	1    0    0    -1
+$EndComp
 Wire Wire Line
 	6450 4300 6600 4300
@@
 L power:GND #PWR012
 U 1 1 619CC4B9
-P 8400 4150
-F 0 "#PWR012" H 8400 3900 50  0001 C CNN
-F 1 "GND" H 8405 3977 50  0000 C CNN
-F 2 "" H 8400 4150 50  0001 C CNN
-F 3 "" H 8400 4150 50  0001 C CNN
-	1    8400 4150
-	1    0    0    -1
-$EndComp
-Wire Wire Line
-	8400 4150 8400 3950
+P 8400 4400
+F 0 "#PWR012" H 8400 4150 50  0001 C CNN
+F 1 "GND" H 8405 4227 50  0000 C CNN
+F 2 "" H 8400 4400 50  0001 C CNN
+F 3 "" H 8400 4400 50  0001 C CNN
+	1    8400 4400
+	1    0    0    -1
+$EndComp
 Wire Wire Line
 	7800 4300 7950 4300
@@
 	7950 3350 7950 3050
 Wire Notes Line
-	3450 4400 3450 2750
-Wire Notes Line
 	3450 2750 8800 2750
-Wire Notes Line
-	8800 2750 8800 4400
-Wire Notes Line
-	8800 4400 3450 4400
-Wire Notes Line
-	4800 4400 4800 2750
-Wire Notes Line
-	6150 4400 6150 2750
-Wire Notes Line
-	7500 4400 7500 2750
 $Comp
 L Transistor_FET:2N7002E Q1
@@
 	1    0    0    -1
 $EndComp
+Wire Wire Line
+	4350 4400 4350 4300
+Connection ~ 4350 4300
+Wire Wire Line
+	4350 4300 4350 3950
+Wire Wire Line
+	3900 4300 4350 4300
+Connection ~ 3900 4300
+Wire Wire Line
+	5700 4400 5700 4300
+Wire Wire Line
+	7050 4400 7050 4300
+Wire Wire Line
+	8400 4400 8400 4300
+Wire Wire Line
+	7950 4300 8400 4300
+Connection ~ 7950 4300
+Connection ~ 8400 4300
+Wire Wire Line
+	8400 4300 8400 3950
+Wire Wire Line
+	6600 4300 7050 4300
+Connection ~ 6600 4300
+Connection ~ 7050 4300
+Wire Wire Line
+	7050 4300 7050 3950
+Wire Wire Line
+	5250 4300 5700 4300
+Connection ~ 5250 4300
+Connection ~ 5700 4300
+Wire Wire Line
+	5700 4300 5700 3950
+Wire Notes Line
+	3450 4650 8800 4650
+Wire Notes Line
+	3450 2750 3450 4650
+Wire Notes Line
+	8800 2750 8800 4650
+Wire Notes Line
+	4800 2750 4800 4650
+Wire Notes Line
+	6150 2750 6150 4650
+Wire Notes Line
+	7500 2750 7500 4650
 $EndSCHEMATC
