File: hardware/nanodrone/nanodrone.kicad_pcb (KiCad board)
At the start: 4 copper layers, 50.8 x 22.9 mm, 22 parts, among them J1 RTR0, J2 RTR1, J3 RTR2, J4 RTR3, Q1 NUD3124LT1G, Q2 NUD3124LT1G, Q3 NUD3124LT1G, Q4 NUD3124LT1G, U1 Feather

Commit message: Rev C
Parts:
- added R11: 25, Resistor_SMD:R_0805_2012Metric_Pad1.20x1.40mm_HandSolder, F.Cu at (161.5, 93.5)
- added R12: 12k, Resistor_SMD:R_0805_2012Metric_Pad1.20x1.40mm_HandSolder, F.Cu at (153.9, 97.3)
- added R13: 4.64k, Resistor_SMD:R_0805_2012Metric_Pad1.20x1.40mm_HandSolder, F.Cu at (153.9, 100.1)
- added R14: 25, Resistor_SMD:R_0805_2012Metric_Pad1.20x1.40mm_HandSolder, F.Cu at (161.5, 98.6)
- Q1, Q2, Q3, Q4: value NUD3124LT1G -> SI2302
- R1: value 10k -> 12k
- R2: value 25 -> 4.64k
- R3: value 10k -> 25
- R4, R8: value 25 -> 12k
- R5: value 10k -> 4.64k
- R7: value 10k -> 100; footprint Resistor_SMD:R_0805_2012Metric_Pad1.20x1.40mm_HandSolder -> Resistor_SMD:R_0805_2012Metric_Pad1.15x1.40mm_HandSolder
- R9: value 100 -> 4.64k; footprint Resistor_SMD:R_0805_2012Metric_Pad1.15x1.40mm_HandSolder -> Resistor_SMD:R_0805_2012Metric_Pad1.20x1.40mm_HandSolder
- moved R6 36.1 mm to (125.5, 98.6), turned to 0 degrees
- moved R5 28.4 mm to (133.1, 100.1), turned to 0 degrees
- moved R7 16.6 mm to (145.5, 102.9), turned to 0 degrees
- moved R9 10.8 mm to (153.9, 95.0)
- moved R8 10.1 mm to (153.9, 92.2), turned to 0 degrees
- moved R1 7.79 mm to (133.1, 92.2), turned to 180 degrees
- moved R2 7.79 mm to (133.1, 95.0)
- moved R4 7.64 mm to (133.1, 97.3), turned to 180 degrees
- moved Q2 3.84 mm to (129.3, 98.6), turned to 180 degrees
- moved Q1 3.82 mm to (129.3, 93.5), turned to 180 degrees
- moved Q3 3.64 mm to (157.7, 93.5), turned to 0 degrees
- moved R3 3.57 mm to (125.5, 93.5)
- moved Q4 3.56 mm to (157.7, 98.6), turned to 0 degrees
- moved D1 1.44 mm to (145.5, 90.4), turned to 0 degrees
- moved D2 1.28 mm to (140.7, 90.4)
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Connections:
- Q1 pad 1: +3V3 -> Net-(Q1-Pad1)
- Q1 pad 2: /rtrctl0 -> GND
- Q2 pad 1: +3V3 -> Net-(Q2-Pad1)
- Q2 pad 2: /rtrctl1 -> GND
- Q3 pad 1: +3V3 -> Net-(Q3-Pad1)
- Q3 pad 2: /rtrctl2 -> GND
- Q4 pad 1: +3V3 -> Net-(Q4-Pad1)
- Q4 pad 2: /rtrctl3 -> GND
- R1 pad 2: /rtrctl0 -> Net-(Q1-Pad1)
- R2 pad 1: +BATT -> Net-(Q1-Pad1)
- R2 pad 2: /rtr0 -> /rtrctl0
- R3 pad 1: +3V3 -> +BATT
- R3 pad 2: /rtrctl1 -> /rtr0
- R4 pad 1: +BATT -> +3V3
- R4 pad 2: /rtr1 -> Net-(Q2-Pad1)
- R5 pad 1: +3V3 -> Net-(Q2-Pad1)
- R5 pad 2: /rtrctl2 -> /rtrctl1
- R6 pad 2: /rtr2 -> /rtr1
- R7 pad 1: +3V3 -> Net-(D1-Pad1)
- R7 pad 2: /rtrctl3 -> GND
- R8 pad 1: +BATT -> +3V3
- R8 pad 2: /rtr3 -> Net-(Q3-Pad1)
- R9 pad 1: Net-(D1-Pad1) -> Net-(Q3-Pad1)
- R9 pad 2: GND -> /rtrctl2
Routing:
- net /rtrctl0: track 47.3 -> 30.6 mm, vias 2 -> 0
- net /rtrctl1: track 43.5 -> 34.8 mm
- net /rtr2: track 12.6 -> 7.11 mm
- net /rtrctl3: track 23.0 -> 17.5 mm
- net /rtr1: track 12.6 -> 7.22 mm
- net /rtr0: track 12.3 -> 7.22 mm
- net /rtr3: track 12.0 -> 7.11 mm
- net Net-(Q2-Pad1): track 0.00 -> 4.84 mm
- net Net-(Q1-Pad1): track 0.00 -> 4.84 mm
- net +3V3: track 11.9 -> 7.19 mm, vias 8 -> 4
- net Net-(Q4-Pad1): track 0.00 -> 4.74 mm
- net Net-(Q3-Pad1): track 0.00 -> 4.74 mm
- net +BATT: track 16.8 -> 12.3 mm
- net /rtrctl2: track 16.9 -> 12.8 mm
- net /dbg1: track 7.19 -> 4.82 mm
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Other:
- board text added: "nanodrone :: RevC nnarain"
- board text removed: "nanodrone :: RevB nnarain"

Commit message: Rev D
Routing:
- net GND: track 5.53 -> 10.1 mm, vias 4 -> 6

Commit message: rev E
Parts:
- removed Q1, Q2, Q3, Q4: SI2302, Package_TO_SOT_SMD:SOT-23
- removed R1, R12, R4, R8: 12k, Resistor_SMD:R_0805_2012Metric_Pad1.20x1.40mm_HandSolder
- removed R11, R14, R3, R6: 25, Resistor_SMD:R_0805_2012Metric_Pad1.20x1.40mm_HandSolder
- removed R13, R2, R5, R9: 4.64k, Resistor_SMD:R_0805_2012Metric_Pad1.20x1.40mm_HandSolder
- added C1: 100nF, Capacitor_SMD:C_0805_2012Metric, F.Cu at (128.9, 96.2)
- added C2: 100nF, Capacitor_SMD:C_0805_2012Metric, F.Cu at (125.7, 93.3)
- added C3: 100nF, Capacitor_SMD:C_0805_2012Metric, F.Cu at (158.1, 95.6)
- added C4: 100nF, Capacitor_SMD:C_0805_2012Metric, F.Cu at (161.3, 98.4)
- added U2: DRV8837, Package_SON:WSON-8-1EP_2x2mm_P0.5mm_EP0.9x1.6mm, F.Cu at (125.7, 95.9)
- added U3: DRV8837, Package_SON:WSON-8-1EP_2x2mm_P0.5mm_EP0.9x1.6mm, F.Cu at (161.3, 95.9)
- R10, R7: footprint Resistor_SMD:R_0805_2012Metric_Pad1.15x1.40mm_HandSolder -> Resistor_SMD:R_0805_2012Metric
- moved R7 1.71 mm to (146.7, 101.6)
- moved R10 1.48 mm to (139.7, 101.6)
- moved D1 1.17 mm to (146.7, 90.2)
- moved D2 1.06 mm to (139.7, 90.2)
Connections:
- J1 pad 1: /rtr0 -> +BATT
- J1 pad 2: GND -> /rtr0
- J2 pad 1: /rtr1 -> +BATT
- J2 pad 2: GND -> /rtr1
- J3 pad 1: /rtr2 -> +BATT
- J3 pad 2: GND -> /rtr2
- J4 pad 1: /rtr3 -> +BATT
- J4 pad 2: GND -> /rtr3
- U1 pad 11: Net-(U1-Pad11) -> unconnected-(U1-Pad11)
- U1 pad 12: Net-(U1-Pad12) -> unconnected-(U1-Pad12)
- U1 pad 13: Net-(U1-Pad13) -> unconnected-(U1-Pad13)
- U1 pad 15: Net-(U1-Pad15) -> unconnected-(U1-Pad15)
- U1 pad 17: Net-(U1-Pad17) -> unconnected-(U1-Pad17)
- U1 pad 18: Net-(U1-Pad18) -> unconnected-(U1-Pad18)
- U1 pad 19: Net-(U1-Pad19) -> unconnected-(U1-Pad19)
- U1 pad 2: Net-(U1-Pad2) -> unconnected-(U1-Pad2)
- U1 pad 20: Net-(U1-Pad20) -> unconnected-(U1-Pad20)
- U1 pad 21: Net-(U1-Pad21) -> unconnected-(U1-Pad21)
- U1 pad 22: Net-(U1-Pad22) -> unconnected-(U1-Pad22)
- U1 pad 23: Net-(U1-Pad23) -> unconnected-(U1-Pad23)
- U1 pad 24: Net-(U1-Pad24) -> unconnected-(U1-Pad24)
- U1 pad 25: Net-(U1-Pad25) -> unconnected-(U1-Pad25)
- U1 pad 26: Net-(U1-Pad26) -> /drv_en1
- U1 pad 27: Net-(U1-Pad27) -> /drv_en2
- U1 pad 28: Net-(U1-Pad28) -> unconnected-(U1-Pad28)
- U1 pad 3: Net-(U1-Pad3) -> unconnected-(U1-Pad3)
- U1 pad 4: Net-(U1-Pad4) -> unconnected-(U1-Pad4)
Routing:
- net /drv_en1: track 0.00 -> 41.4 mm, vias 0 -> 2
- net /drv_en2: track 0.00 -> 16.8 mm, vias 0 -> 2
- net /rtr3: track 7.11 -> 22.4 mm
- net +BATT: track 12.3 -> 25.7 mm
- net /rtrctl0: track 30.6 -> 44.0 mm, vias 0 -> 2
- net GND: track 10.1 -> 17.2 mm, vias 6 -> 4
- net Net-(Q2-Pad1): track 4.84 -> 0.00 mm
- net Net-(Q1-Pad1): track 4.84 -> 0.00 mm
- net /rtr2: track 7.11 -> 11.9 mm, vias 0 -> 2
- net Net-(Q4-Pad1): track 4.74 -> 0.00 mm
- net Net-(Q3-Pad1): track 4.74 -> 0.00 mm
- net /rtrctl2: track 12.8 -> 17.3 mm, vias 1 -> 0
- net /rtr1: track 7.22 -> 11.4 mm
- net /rtrctl1: track 34.8 -> 38.1 mm
- net /rtrctl3: track 17.5 -> 20.3 mm, vias 1 -> 0
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- added copper zone on In2.Cu, net +3V3
- added copper zone on In2.Cu, net +BATT
- added copper zone on In1.Cu, net GND
- removed copper zone on PWR, net +3V3
- removed copper zone on PWR, net +BATT
- removed copper zone on GND, net GND
Other:
- net class Default removed
- board text added: "nanodrone :: RevE nnarain"
- board text removed: "nanodrone :: RevC nnarain"
