File: hardware/nanodrone/nanodrone.kicad_sch (KiCad schematic)
At the start: 15 parts, among them J1 RTR0, J2 RTR1, J3 RTR2, J4 RTR3, U1 Feather, U2 DRV8837, U3 DRV8837

Commit message: kibot bom config
Parts:
- D1: LCSC (none) -> C434432; LCSC Part Number C434432 -> (none)
- D2: LCSC (none) -> C434432; LSCS Part Number C434432 -> (none)
- R10, R7: LCSC (none) -> C17408; LCSC Part Number C17408 -> (none)
Changed lines of the file:
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@@
       (effects (font (size 1.27 1.27)) hide)
     )
-    (property "LCSC Part Number" "C434432" (id 5) (at 135.89 121.92 90)
+    (property "LCSC" "C434432" (id 5) (at 135.89 121.92 90)
       (effects (font (size 1.27 1.27)) hide)
     )
@@
       (effects (font (size 1.27 1.27)) hide)
     )
-    (property "LSCS Part Number" "C434432" (id 5) (at 147.32 121.92 90)
+    (property "LCSC" "C434432" (id 5) (at 147.32 121.92 90)
       (effects (font (size 1.27 1.27)) hide)
     )
@@
       (effects (font (size 1.27 1.27)) hide)
     )
-    (property "LCSC Part Number" "C17408" (id 5) (at 135.89 132.08 0)
+    (property "LCSC" "C17408" (id 5) (at 135.89 132.08 0)
       (effects (font (size 1.27 1.27)) hide)
     )
@@
       (effects (font (size 1.27 1.27)) hide)
     )
-    (property "LCSC Part Number" "C17408" (id 5) (at 147.32 132.08 0)
+    (property "LCSC" "C17408" (id 5) (at 147.32 132.08 0)
       (effects (font (size 1.27 1.27)) hide)
     )
